File: design.kicad_sch (KiCad schematic)
At the start: 0 parts

Commit message: SCH Add initial design
Parts:
- added C?: 0-50pF, Capacitor_SMD:C_0805_2012Metric, symbol Device:C_Small
- added C? (x3): C_Small, symbol Device:C_Small
- added C?: 0.1uF, Capacitor_SMD:C_0805_2012Metric, symbol Device:C_Small
- added C?: 1uF, symbol Device:C_Small
- added C?: 100nF, Capacitor_SMD:C_0805_2012Metric, symbol Device:C_Small
- added C?: 10uF, Capacitor_SMD:C_0805_2012Metric, symbol Device:C_Small
- added JP?: AHLB, Jumper:SolderJumper-2_P1.3mm_Bridged_RoundedPad1.0x1.5mm, symbol Jumper:Jumper_2_Bridged
- added JP?: TOG, Jumper:SolderJumper-2_P1.3mm_Open_RoundedPad1.0x1.5mm, symbol Jumper:Jumper_2_Open
- added L?: L_Small, symbol Device:L_Small
- added R? (x2): R_Small, symbol Device:R_Small
- added R?: 10K, symbol Device:R_Small
- added U?: AP3015, Package_TO_SOT_SMD:SOT-23-5, symbol Regulator_Switching:AP3012
- added U?: TCK127BG,LF, symbol Power_Management_custom:TCK127BG,LF
- added U?: ESP32-C3-WROOM-02-N4, MODULE_ESP32-C3-WROOM-02-H4, symbol MCU_Espressif_custom:ESP32-C3-WROOM-02-N4
- added U?: TTP223, Package_TO_SOT_SMD:SOT-23-6_Handsoldering, symbol LEDs:TTP223
Connections:
- new net: R?.1, R?.2, U?.3 (FB)
- new net: C?.1, L?.1, U?.4 (~{SHDN}), U?.5 (IN), U?.A1 (VOUT)
- new net: C?.1, R?.2, U?.2 (EN)
- new net: JP?.1 (A), U?.4 (AHLB)
- new net: JP?.1 (A), U?.6 (TOG)
- new net GND: C?.2, C?.2, C?.2, C?.2, C?.2, C?.2, C?.2, C?.2, R?.2, U?.19 (GND), U?.2 (GND), U?.2 (GND), U?.20 (GND), U?.21 (GND), U?.22 (GND), U?.23 (GND), U?.24 (GND), U?.25 (GND), U?.26 (GND), U?.27 (GND), U?.28 (GND), U?.29 (GND), U?.30 (GND), U?.31 (GND), U?.32 (GND), U?.33 (GND), U?.34 (GND), U?.35 (GND), U?.36 (GND), U?.37 (GND), U?.38 (GND), U?.39 (GND), U?.9 (GND), U?.B1 (GND)
- new net PWR_control: U?.B2 (Control)
- new net VCC: C?.1, C?.1, C?.1, C?.1, C?.1, JP?.2 (B), JP?.2 (B), L?.2, R?.1, R?.1, U?.1 (3V3), U?.1 (SW), U?.5 (VCC)
- new net Vbat: U?.A2 (VIN)
- new net touch_point: C?.1, U?.3 (I)
- new net touch_state: U?.1 (Q)
Other:
- note added: "No intenal LDO - feed with fixed valtage between 2-5.5V"
- note added: "Touch IC TTP223"
