File: design.kicad_sch (KiCad schematic)
At the start: 18 parts

Commit message: Update design.kicad_sch
Parts:
- U1: renamed from U?; value TCK127BG,LF -> TCK127BG
- gave numbers to parts that had none: 17

Commit message: iBom fix (#5)
* enable iBOM action

* add footprints

* Update design.kicad_pcb

* Update design.kicad_sch

* PCB outline
Parts:
- C1, C2, C3, C4: footprint (none) -> Capacitor_SMD:C_0805_2012Metric
- L1: footprint (none) -> Inductor_SMD:L_TracoPower_TCK-047_5.2x5.8mm
- R1, R2, R3: footprint (none) -> Resistor_SMD:R_0805_2012Metric
- U1: footprint (none) -> Package_BGA_custom:Toshiba_WCSP4G
- U3: footprint MODULE_ESP32-C3-WROOM-02-H4 -> MCU_Espressif_custom:MODULE_ESP32-C3-WROOM-02-H4
Changed lines of the file:
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@@
       (effects (font (size 1.27 1.27)) (justify left))
     )
-    (property "Footprint" "" (id 2) (at 120.65 62.865 0)
+    (property "Footprint" "Resistor_SMD:R_0805_2012Metric" (id 2) (at 120.65 62.865 0)
       (effects (font (size 1.27 1.27)) hide)
     )
@@
     (property "Reference" "U1" (id 0) (at 45.72 27.94 0))
     (property "Value" "TCK127BG" (id 1) (at 45.72 30.48 0))
-    (property "Footprint" "" (id 2) (at 45.72 38.735 0)
+    (property "Footprint" "Package_BGA_custom:Toshiba_WCSP4G" (id 2) (at 45.72 38.735 0)
       (effects (font (size 1.27 1.27)) hide)
     )
@@
     (pin "B1")
     (pin "B2")
+    (pin "A1-UB")
+    (pin "A2-UB")
+    (pin "B1-UB")
+    (pin "B2-UB")
+    (pin "A1-UC")
+    (pin "A2-UC")
+    (pin "B1-UC")
+    (pin "B2-UC")
+    (pin "A1-UD")
+    (pin "A2-UD")
+    (pin "B1-UD")
+    (pin "B2-UD")
   )
   (symbol (lib_id "Device:R_Small") (at 120.65 41.91 0) (unit 1)
@@
       (effects (font (size 1.27 1.27)) (justify left))
     )
-    (property "Footprint" "" (id 2) (at 120.65 41.91 0)
+    (property "Footprint" "Resistor_SMD:R_0805_2012Metric" (id 2) (at 120.65 41.91 0)
       (effects (font (size 1.27 1.27)) hide)
     )
@@
       (effects (font (size 1.27 1.27)) (justify left))
     )
-    (property "Footprint" "" (id 2) (at 189.865 99.695 0)
+    (property "Footprint" "Resistor_SMD:R_0805_2012Metric" (id 2) (at 189.865 99.695 0)
       (effects (font (size 1.27 1.27)) hide)
     )
@@
     (property "Reference" "U3" (id 0) (at 219.71 94.615 0))
     (property "Value" "ESP32-C3-WROOM-02-N4" (id 1) (at 219.71 97.155 0))
-    (property "Footprint" "MODULE_ESP32-C3-WROOM-02-H4" (id 2) (at 219.71 120.65 0)
+    (property "Footprint" "MCU_Espressif_custom:MODULE_ESP32-C3-WROOM-02-H4" (id 2) (at 219.71 120.65 0)
       (effects (font (size 1.27 1.27)) (justify left bottom) hide)
     )
@@
     (property "Reference" "L1" (id 0) (at 103.505 31.115 90))
     (property "Value" "L_Small" (id 1) (at 103.505 33.655 90))
-    (property "Footprint" "" (id 2) (at 103.505 36.195 0)
+    (property "Footprint" "Inductor_SMD:L_TracoPower_TCK-047_5.2x5.8mm" (id 2) (at 103.505 36.195 0)
       (effects (font (size 1.27 1.27)) hide)
     )
@@
       (effects (font (size 1.27 1.27)) (justify left))
     )
-    (property "Footprint" "" (id 2) (at 144.145 50.165 0)
+    (property "Footprint" "Capacitor_SMD:C_0805_2012Metric" (id 2) (at 144.145 50.165 0)
       (effects (font (size 1.27 1.27)) hide)
     )
@@
       (effects (font (size 1.27 1.27)) (justify left))
     )
-    (property "Footprint" "" (id 2) (at 180.975 107.95 0)
+    (property "Footprint" "Capacitor_SMD:C_0805_2012Metric" (id 2) (at 180.975 107.95 0)
       (effects (font (size 1.27 1.27)) hide)
     )
@@
       (effects (font (size 1.27 1.27)) (justify left))
     )
-    (property "Footprint" "" (id 2) (at 132.08 46.355 0)
+    (property "Footprint" "Capacitor_SMD:C_0805_2012Metric" (id 2) (at 132.08 46.355 0)
       (effects (font (size 1.27 1.27)) hide)
     )
@@
       (effects (font (size 1.27 1.27)) (justify left))
     )
-    (property "Footprint" "" (id 2) (at 71.755 49.53 0)
+    (property "Footprint" "Capacitor_SMD:C_0805_2012Metric" (id 2) (at 71.755 49.53 0)
       (effects (font (size 1.27 1.27)) hide)
     )
@@
     )
     (path "/e25ae11e-2d4c-4183-bf19-5432810f78c3"
-      (reference "C1") (unit 1) (value "C_Small") (footprint "")
+      (reference "C1") (unit 1) (value "C_Small") (footprint "Capacitor_SMD:C_0805_2012Metric")
     )
     (path "/f0307fb3-2ec2-4eb2-8563-0e6b4d6f1e24"
-      (reference "C2") (unit 1) (value "C_Small") (footprint "")
+      (reference "C2") (unit 1) (value "C_Small") (footprint "Capacitor_SMD:C_0805_2012Metric")
     )
     (path "/5c65d500-5747-4144-b0ce-e8ba6f5cbe3b"
-      (reference "C3") (unit 1) (value "C_Small") (footprint "")
+      (reference "C3") (unit 1) (value "C_Small") (footprint "Capacitor_SMD:C_0805_2012Metric")
     )
     (path "/b15030b4-a6e9-4f45-b2c0-ca7b53cc6121"
-      (reference "C4") (unit 1) (value "1uF") (footprint "")
+      (reference "C4") (unit 1) (value "1uF") (footprint "Capacitor_SMD:C_0805_2012Metric")
     )
     (path "/e44e7433-fc25-4571-b40e-1763b14d59ef"
@@
     )
     (path "/50e6e7dd-73e0-4324-bc63-c9a8c6c1e423"
-      (reference "L1") (unit 1) (value "L_Small") (footprint "")
+      (reference "L1") (unit 1) (value "L_Small") (footprint "Inductor_SMD:L_TracoPower_TCK-047_5.2x5.8mm")
     )
     (path "/28ef594d-4759-4905-9812-be4944849ce8"
-      (reference "R1") (unit 1) (value "R_Small") (footprint "")
+      (reference "R1") (unit 1) (value "R_Small") (footprint "Resistor_SMD:R_0805_2012Metric")
     )
     (path "/197c587c-0905-4e20-a7d9-9496799e8039"
-      (reference "R2") (unit 1) (value "R_Small") (footprint "")
+      (reference "R2") (unit 1) (value "R_Small") (footprint "Resistor_SMD:R_0805_2012Metric")
     )
     (path "/29c9952d-0114-4f73-9078-7f0aa87ca54b"
-      (reference "R3") (unit 1) (value "10K") (footprint "")
+      (reference "R3") (unit 1) (value "10K") (footprint "Resistor_SMD:R_0805_2012Metric")
     )
     (path "/25ada721-670a-4020-ae0b-77410c4e375a"
-      (reference "U1") (unit 1) (value "TCK127BG") (footprint "")
+      (reference "U1") (unit 1) (value "TCK127BG") (footprint "Package_BGA_custom:Toshiba_WCSP4G")
     )
     (path "/0f42af37-45d6-4a55-bb59-732500a7cdbf"
@@
     )
     (path "/2f9221d0-9237-419d-a405-ed6293d81ca2"
-      (reference "U3") (unit 1) (value "ESP32-C3-WROOM-02-N4") (footprint "MODULE_ESP32-C3-WROOM-02-H4")
+      (reference "U3") (unit 1) (value "ESP32-C3-WROOM-02-N4") (footprint "MCU_Espressif_custom:MODULE_ESP32-C3-WROOM-02-H4")
     )
     (path "/e8885089-96ba-4731-a75f-c51ec6dc2615"
