File: design.kicad_pcb (KiCad board)
At the start: 2 copper layers, 0 parts

Commit message: iBom fix (#5)
* enable iBOM action

* add footprints

* Update design.kicad_pcb

* Update design.kicad_sch

* PCB outline
Parts:
- added C1: C_Small, Capacitor_SMD:C_0805_2012Metric, F.Cu at (141.0, 81.0)
- added C2: C_Small, Capacitor_SMD:C_0805_2012Metric, F.Cu at (120.2, 102.5)
- added C3: C_Small, Capacitor_SMD:C_0805_2012Metric, F.Cu at (128.3, 92.7)
- added C4: 1uF, Capacitor_SMD:C_0805_2012Metric, F.Cu at (134.2, 88.0)
- added C5: 10uF, Capacitor_SMD:C_0805_2012Metric, F.Cu at (128.3, 95.7)
- added C6: 0.1uF, Capacitor_SMD:C_0805_2012Metric, F.Cu at (111.3, 102.5)
- added C7: 100nF, Capacitor_SMD:C_0805_2012Metric, F.Cu at (115.7, 102.5)
- added C8: 0-50pF, Capacitor_SMD:C_0805_2012Metric, F.Cu at (106.8, 102.5)
- added JP1: TOG, Jumper:SolderJumper-2_P1.3mm_Open_RoundedPad1.0x1.5mm, F.Cu at (128.2, 99.0)
- added JP2: AHLB, Jumper:SolderJumper-2_P1.3mm_Bridged_RoundedPad1.0x1.5mm, F.Cu at (145.4, 81.3)
- added L1: L_Small, Inductor_SMD:L_TracoPower_TCK-047_5.2x5.8mm, F.Cu at (129.8, 83.0)
- added R1: R_Small, Resistor_SMD:R_0805_2012Metric, F.Cu at (141.0, 84.0)
- added R2: R_Small, Resistor_SMD:R_0805_2012Metric, F.Cu at (132.7, 92.7)
- added R3: 10K, Resistor_SMD:R_0805_2012Metric, F.Cu at (138.6, 86.9)
- added U1: TCK127BG, Package_BGA_custom:Toshiba_WCSP4G, F.Cu at (136.0, 98.0)
- added U2: AP3015, Package_TO_SOT_SMD:SOT-23-5, F.Cu at (136.2, 81.7)
- added U3: ESP32-C3-WROOM-02-N4, MCU_Espressif_custom:MODULE_ESP32-C3-WROOM-02-H4, F.Cu at (115.8, 90.3)
- added U4: TTP223, Package_TO_SOT_SMD:SOT-23-6_Handsoldering, F.Cu at (129.0, 88.9)
Other:
- board outline added: 55.5 x 30.5 mm

Commit message: PCB scramble
Parts:
- added C10: 0-50pF, Capacitor_SMD:C_0805_2012Metric, F.Cu at (109.2, 82.1)
- added C11: 0-50pF, Capacitor_SMD:C_0805_2012Metric, F.Cu at (130.9, 81.8)
- added C9: 100nF, Capacitor_SMD:C_0805_2012Metric, F.Cu at (130.9, 74.5)
- added D1: SS14, Diode_SMD:D_SMA, F.Cu at (119.0, 55.7)
- added D2: D_Small, Diode_SMD:D_SOD-323, F.Cu at (132.8, 58.2)
- added D3: LED, LED_SMD:LED_0603_1608Metric, F.Cu at (99.0, 51.8)
- added D4: LED, LED_SMD:LED_0603_1608Metric, F.Cu at (138.9, 48.4)
- added D5: LED, LED_SMD:LED_0603_1608Metric, F.Cu at (118.2, 48.0)
- added D6: D_Small, Diode_SMD:D_SOD-323, F.Cu at (126.2, 75.8)
- added D7: D_Small, Diode_SMD:D_SOD-323, F.Cu at (104.8, 75.8)
- added H1: MountingHole, MountingHole:MountingHole_3.2mm_M3, F.Cu at (266.5, 41.5)
- added H2: MountingHole, MountingHole:MountingHole_3.2mm_M3, F.Cu at (265.0, 52.0)
- added H3: MountingHole, MountingHole:MountingHole_3.2mm_M3, F.Cu at (265.0, 62.5)
- added H4: MountingHole, MountingHole:MountingHole_3.2mm_M3, F.Cu at (266.0, 30.0)
- added J2: Programming, Connector_PinHeader_2.54mm:PinHeader_1x04_P2.54mm_Vertical, F.Cu at (135.0, 48.0)
- added J3: HRO_TYPE-C-31-M-12, Connector_USB:USB_C_Receptacle_HRO_TYPE-C-31-M-12, F.Cu at (143.0, 39.0)
- added JP3: SHDN-Control, Jumper:SolderJumper-3_P1.3mm_Bridged12_RoundedPad1.0x1.5mm_NumberLabels, F.Cu at (114.8, 66.7)
- added JP4: TOG, Jumper:SolderJumper-2_P1.3mm_Open_RoundedPad1.0x1.5mm, F.Cu at (114.8, 76.6)
- added JP5: TOG, Jumper:SolderJumper-2_P1.3mm_Open_RoundedPad1.0x1.5mm, F.Cu at (136.8, 76.4)
- added JP6: AHLB, Jumper:SolderJumper-2_P1.3mm_Open_RoundedPad1.0x1.5mm, F.Cu at (114.8, 79.2)
- added JP7: AHLB, Jumper:SolderJumper-2_P1.3mm_Open_RoundedPad1.0x1.5mm, F.Cu at (136.8, 79.0)
- added R10: 470, Resistor_SMD:R_0805_2012Metric, F.Cu at (121.8, 48.0)
- added R11: 10K, Resistor_SMD:R_0805_2012Metric, F.Cu at (135.5, 34.6)
- added R12: 10K, Resistor_SMD:R_0805_2012Metric, F.Cu at (107.0, 41.0)
- added R4: 5.1k, Resistor_SMD:R_0805_2012Metric, F.Cu at (141.0, 45.5)
- added R5: 10K, Resistor_SMD:R_0805_2012Metric, F.Cu at (137.2, 58.2)
- added R6: 10K, Resistor_SMD:R_0805_2012Metric, F.Cu at (107.5, 34.2)
- added R7: 10K, Resistor_SMD:R_0805_2012Metric, F.Cu at (132.8, 31.7)
- added R8: 330, Resistor_SMD:R_0805_2012Metric, F.Cu at (99.0, 55.4)
- added R9: 330, Resistor_SMD:R_0805_2012Metric, F.Cu at (140.5, 51.2)
- added SW1: SW_Push, Button_Switch_SMD:SW_SPST_EVPBF, F.Cu at (135.8, 63.0)
- added SW2: EN, Button_Switch_SMD:SW_SPST_EVPBF, F.Cu at (99.4, 34.8)
- added SW3: IO0, Button_Switch_SMD:SW_SPST_EVPBF, F.Cu at (99.4, 43.9)
- added TP1: GND, TestPoint:TestPoint_Pad_D2.5mm, F.Cu at (143.0, 48.8)
- added TP2: VCC, TestPoint:TestPoint_Pad_D2.5mm, F.Cu at (143.0, 53.9)
- added TP3: +3.3V, TestPoint:TestPoint_Pad_D2.5mm, F.Cu at (109.2, 51.4)
- added U5: TTP223, Package_TO_SOT_SMD:SOT-23-6_Handsoldering, F.Cu at (130.9, 77.8)
- C2: value C_Small -> 4.7uF
- C3: value C_Small -> 10pF
- C4: value 1uF -> 20uF
- C7: value 100nF -> 1uF
- C8: value 0-50pF -> 100nF
- JP1: value TOG -> Switch_jump
- JP2: value AHLB -> Reg_jump; footprint Jumper:SolderJumper-2_P1.3mm_Bridged_RoundedPad1.0x1.5mm -> Jumper:SolderJumper-2_P1.3mm_Open_RoundedPad1.0x1.5mm
- L1: value L_Small -> 10uH
- R1: value R_Small -> 1M
- R2: value R_Small -> 600k
- R3: value 10K -> 5.1k
- moved C6 71.1 mm to (108.5, 31.5), turned to 90 degrees
- moved C5 67.9 mm to (106.2, 31.5), turned to 90 degrees
- moved C7 66.1 mm to (107.2, 37.0), turned to -90 degrees
- moved U3 54.9 mm to (120.0, 35.5)
- moved R3 54.5 mm to (141.0, 32.5)
- moved JP1 46.0 mm to (127.8, 53.0), turned to 180 degrees
- moved U1 43.8 mm to (131.9, 54.4)
- moved C4 40.9 mm to (115.4, 51.7), turned to 180 degrees
- moved C3 40.6 mm to (115.4, 54.2), turned to 180 degrees
- moved R1 37.7 mm to (114.0, 57.7), turned to -90 degrees
- moved R2 36.2 mm to (114.0, 61.7), turned to -90 degrees
- moved C2 35.9 mm to (119.5, 66.7), turned to -90 degrees
- moved JP2 35.7 mm to (123.6, 53.0), turned to 180 degrees
- moved C1 31.0 mm to (131.9, 51.4), turned to 180 degrees
- moved C8 28.3 mm to (109.2, 74.3), turned to 180 degrees
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Connections:
- net Net-(R1-Pad2) renamed /FB
- C1 pad 1: VCC -> Vbat
- C2 pad 1: Net-(C2-Pad1) -> /In
- C3 pad 1: VCC -> +3.3V
- C4 pad 1: Net-(C4-Pad1) -> +3.3V
- C5 pad 1: VCC -> +3.3V
- C6 pad 1: VCC -> +3.3V
- C7 pad 1: VCC -> /EN
- C8 pad 1: touch_point -> Vbat
- JP1 pad 1: Net-(JP1-Pad1) -> Vbat
- JP1 pad 2: VCC -> /In
- JP2 pad 1: Net-(JP2-Pad1) -> /In
- JP2 pad 2: VCC -> +3.3V
- L1 pad 1: Net-(C2-Pad1) -> /In
- L1 pad 2: VCC -> /SW
- R1 pad 1: VCC -> +3.3V
- R3 pad 1: VCC -> GND
- R3 pad 2: Net-(C4-Pad1) -> /CC2
- U1 pad A1: Net-(C2-Pad1) -> /In
- U1 pad B2: PWR_control -> IO6
- U2 pad 1: VCC -> /SW
- U2 pad 4: Net-(C2-Pad1) -> /SHDN
- U2 pad 5: Net-(C2-Pad1) -> /In
- U3 pad 1: VCC -> +3.3V
- U3 pad 10: unconnected-(U3-Pad10) -> IO10
- U3 pad 11: unconnected-(U3-Pad11) -> MCU_RX
- U3 pad 12: unconnected-(U3-Pad12) -> MCU_TX
- U3 pad 13: unconnected-(U3-Pad13) -> D-
- U3 pad 14: unconnected-(U3-Pad14) -> D+
- U3 pad 15: unconnected-(U3-Pad15) -> IO3
- U3 pad 16: unconnected-(U3-Pad16) -> IO2
- U3 pad 17: unconnected-(U3-Pad17) -> IO1
- U3 pad 18: unconnected-(U3-Pad18) -> /IO0
- U3 pad 2: Net-(C4-Pad1) -> /EN
- U3 pad 3: unconnected-(U3-Pad3) -> IO4
- U3 pad 4: unconnected-(U3-Pad4) -> IO5
- U3 pad 5: unconnected-(U3-Pad5) -> IO6
- U3 pad 6: unconnected-(U3-Pad6) -> IO7
- U3 pad 7: unconnected-(U3-Pad7) -> IO8
- U3 pad 8: unconnected-(U3-Pad8) -> IO9
- U4 pad 1: touch_state -> IO5
- U4 pad 3: touch_point -> touch_point_1
- U4 pad 4: Net-(JP2-Pad1) -> Net-(U4-Pad4)
- U4 pad 5: VCC -> Vbat
- U4 pad 6: Net-(JP1-Pad1) -> Net-(JP4-Pad1)
Routing:
- net Vbat: track 0.00 -> 117.6 mm, vias 0 -> 7
- net +3.3V: track 0.00 -> 110.7 mm
- net IO6: track 0.00 -> 94.8 mm, vias 0 -> 3
- net IO4: track 0.00 -> 57.2 mm, vias 0 -> 2
- net IO5: track 0.00 -> 49.4 mm, vias 0 -> 2
- net /IO0: track 0.00 -> 40.8 mm, vias 0 -> 2
- net /In: track 0.00 -> 27.0 mm
- net GND: track 0.00 -> 22.0 mm, vias 0 -> 8
- net Net-(R5-Pad2): track 0.00 -> 18.8 mm
- net IO7: track 0.00 -> 18.3 mm, vias 0 -> 2
- net /EN: track 0.00 -> 17.5 mm, vias 0 -> 2
- net D+: track 0.00 -> 12.8 mm
- net D-: track 0.00 -> 10.3 mm
- net /CC1: track 0.00 -> 9.75 mm
- net /control: track 0.00 -> 8.95 mm
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- added copper zone on F.Cu, net /In
- added copper zone on B.Cu, net GND
- added copper zone on F.Cu, net GND
- added copper zone on B.Cu, net Vbat
- added copper zone on B.Cu, net touch_point_1
- added copper zone on B.Cu, net touch_point_2
Other:
- board size 55.5 x 30.5 mm -> 51.7 x 59.7 mm

Commit message: Update design.kicad_pcb
Parts:
- moved H3 161.7 mm to (119.2, 132.4)
- moved H2 146.8 mm to (119.2, 69.4)
- moved H4 145.1 mm to (163.2, 132.4)
- moved H1 107.0 mm to (163.2, 69.4)
- moved C10 48.0 mm to (130.2, 125.3)
- moved C11 48.0 mm to (151.9, 125.0)
- moved C2 48.0 mm to (140.5, 109.9)
- moved C3 48.0 mm to (136.4, 97.4)
- moved C4 48.0 mm to (136.4, 94.9)
- moved C5 48.0 mm to (127.2, 74.7)
- moved C6 48.0 mm to (129.5, 74.7)
- moved C7 48.0 mm to (128.2, 80.2)
- moved C8 48.0 mm to (130.2, 117.5)
- moved C9 48.0 mm to (151.9, 117.8)
- moved D1 48.0 mm to (140.0, 98.9)
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Routing:
- net GND: track 22.0 -> 55.0 mm, vias 8 -> 13
- net IO6: track 94.8 -> 99.2 mm
- net D-: track 10.3 -> 13.6 mm
- net /IO0: track 40.8 -> 41.8 mm
- net /EN: track 17.5 -> 18.4 mm
Other:
- board size 51.7 x 59.7 mm -> 54 x 71.1 mm
- board text added: "Touch 1"
- board text added: "Touch 2"
